Commit message: change 1

File: kinova-ros-master/kinova_description/urdf/j2n6s300_standalone.xacro (robot description, xacro)
@@ -26,8 +26,8 @@
     <child link="camera_rack_link" />
     <parent link="j2n6s300_link_6" />
-    <origin xyz="0 0 0.007" rpy="0 0 3.14159" />
+    <origin xyz="0 0 0.007" rpy="0 0 0" />
   </joint>
   <link name="camera_rack_link">
-    <!--visual>
+    <visual>
       <origin
         xyz="0 0 0"
@@ -42,5 +42,5 @@
           rgba="0.792156862745098 0.819607843137255 0.933333333333333 1" />
       </material>
-    </visual-->
+    </visual>
   </link>
   <joint name="camera_joint" type="fixed">
@@ -50,5 +50,5 @@
   </joint>
   <link name="camera_link">
-    <!--visual>
+    <visual>
       <origin
         xyz="0 0 0"
@@ -63,5 +63,5 @@
           rgba="0.792156862745098 0.819607843137255 0.933333333333333 1" />
       </material>
-    </visual-->
+    </visual>
   </link>
   <xacro:property name="robot_root" value="root" />

Commit message: to windows

File: kinova-ros-master/kinova_description/urdf/j2n6s300_standalone.xacro (robot description, xacro)
@@ -29,5 +29,5 @@
   </joint>
   <link name="camera_rack_link">
-    <visual>
+    <!--visual>
       <origin
         xyz="0 0 0"
@@ -42,5 +42,5 @@
           rgba="0.792156862745098 0.819607843137255 0.933333333333333 1" />
       </material>
-    </visual>
+    </visual-->
   </link>
   <joint name="camera_joint" type="fixed">
@@ -50,5 +50,5 @@
   </joint>
   <link name="camera_link">
-    <visual>
+    <!--visual>
       <origin
         xyz="0 0 0"
@@ -63,5 +63,5 @@
           rgba="0.792156862745098 0.819607843137255 0.933333333333333 1" />
       </material>
-    </visual>
+    </visual-->
   </link>
   <xacro:property name="robot_root" value="root" />

Commit message: open door v1 and has a problem

File: kinova-ros-master/kinova_description/urdf/j2n6s300_standalone.xacro (robot description, xacro)
@@ -26,5 +26,5 @@
     <child link="camera_rack_link" />
     <parent link="j2n6s300_link_6" />
-    <origin xyz="0 0 0.007" rpy="0 0 0" />
+    <origin xyz="0 0 0.007" rpy="0 0 3.14159" />
   </joint>
   <link name="camera_rack_link">
